Commit message: switch from .obj to .stl for mujoco compile, add generated mjcf file

File: gym/envs/robotics/assets/panda/panda_urdf/panda.urdf (robot description, URDF)
Before this commit: robot panda, 12 links, 11 joints
Links:
- link panda_hand: geometry collision mesh filename=package://Panda/meshes/collision/hand.stl; visual mesh filename=package://Panda/meshes/collision/hand.stl
- link panda_leftfinger: geometry collision mesh filename=package://Panda/meshes/collision/finger.stl; visual mesh filename=package://Panda/meshes/collision/finger.stl
- link panda_link0: geometry collision mesh filename=package://Panda/meshes/collision/link0.stl; visual mesh filename=package://Panda/meshes/collision/link0.stl
- link panda_link1: geometry collision mesh filename=package://Panda/meshes/collision/link1.stl; visual mesh filename=package://Panda/meshes/collision/link1.stl
- link panda_link2: geometry collision mesh filename=package://Panda/meshes/collision/link2.stl; visual mesh filename=package://Panda/meshes/collision/link2.stl
- link panda_link3: geometry collision mesh filename=package://Panda/meshes/collision/link3.stl; visual mesh filename=package://Panda/meshes/collision/link3.stl
- link panda_link4: geometry collision mesh filename=package://Panda/meshes/collision/link4.stl; visual mesh filename=package://Panda/meshes/collision/link4.stl
- link panda_link5: geometry collision mesh filename=package://Panda/meshes/collision/link5.stl; visual mesh filename=package://Panda/meshes/collision/link5.stl
- link panda_link6: geometry collision mesh filename=package://Panda/meshes/collision/link6.stl; visual mesh filename=package://Panda/meshes/collision/link6.stl
- link panda_link7: geometry collision mesh filename=package://Panda/meshes/collision/link7.stl; visual mesh filename=package://Panda/meshes/collision/link7.stl
- link panda_rightfinger: geometry collision mesh filename=package://Panda/meshes/collision/finger.stl; visual mesh filename=package://Panda/meshes/collision/finger.stl
